Commit message: Add files via upload

File: robot_siad7n/urdf/robot_siad7n.urdf (robot description, URDF)
Before this commit: robot robot_siad7n, 8 links, 7 joints
Links:
- link base_link: mass 9.5605 -> 9.5604593531081
Joints:
- joint joint_1: origin xyz=0 0 0.1265 rpy=1.5708 0 0 -> xyz=0 0 0.1265 rpy=1.5707963267949 0 0
- joint joint_2: origin xyz=0 0.298 0 rpy=0 0 0 -> xyz=0 0.297999999999997 0 rpy=0 0 0
- joint joint_3: limit lower=0.32 upper=0.32 effort=500 velocity=10 -> lower=0 upper=0.32 effort=500 velocity=10
- joint joint_5: origin xyz=0.12764 -0.29297 -0.021311 rpy=-1.5708 1.5276 1.5708 -> xyz=0.127639785374671 -0.292970498838426 -0.0213107930928151 rpy=-1.5707963267949 1.52758843931606 1.5707963267949
- joint joint_6: origin xyz=-0.091413 0.18088 0 rpy=3.1416 0 -3.1416 -> xyz=-0.0914130137207118 0.180882427216801 0 rpy=3.14159265358979 0 -3.14159265358979
- joint joint_7: axis 0 0.99907 -0.043194 -> 0 0.999066684445606 -0.0431944444444357; origin xyz=0 0.1622 0.01686 rpy=0.043208 1.5708 0 -> xyz=0 0.1621961599513 0.0168602146253252 rpy=0.0432078874788314 1.5707963267949 0

Commit message: Add files via upload

File: robot_siad7n/urdf/robot_siad7n.urdf (robot description, URDF)
Before this commit: robot robot_siad7n, 8 links, 7 joints
Links:
- removed link end_efector
- added link EF, mass 9.59762719689291E-05; collision mesh filename=package://robot_siad7n/meshes/EF.STL; visual mesh filename=package://robot_siad7n/meshes/EF.STL
- link base_link: mass 9.5604593531081 -> 9.5605
- link link_1: mass 11.7569497464344 -> 0.0117569497463589
- link link_2: mass 10.0552877935453 -> 10.0552877935848
- link link_3: mass 8.43890800694608 -> 0.00843890832225914
- link link_4: mass 6.45549495463595 -> 6.45548607858182
- link link_5: mass 2.87980693010728 -> 0.00287980676910192
- link link_6: mass 2.01842022888389 -> 0.0020184
Joints:
- removed joint joint_3
- added joint join_3: type prismatic, parent link_2, child link_3, origin xyz=3.4347E-05 0.3019 0.265 rpy=0 0 3.1416, axis 0 1 0, limit lower=0 upper=0.32 effort=100 velocity=10
- joint joint_1: origin xyz=0 0 0.1265 rpy=1.5707963267949 0 0 -> xyz=0 0 0.1175 rpy=1.5708 0 0
- joint joint_2: origin xyz=0 0.297999999999997 0 rpy=0 0 0 -> xyz=0 0.298 0 rpy=0 0 0
- joint joint_4: axis 0 0.043194 -0.99907 -> 0 0 1; limit lower=-3.1416 upper=0 effort=0 velocity=0 -> lower=-1.3963 upper=4.5379 effort=0 velocity=0; origin xyz=-0.12061 0.2426 -0.0092049 rpy=3.0984 0 1.5708 -> xyz=0 -0.2426 0 rpy=3.1416 0 -1.5708
- joint joint_5: origin xyz=0.127639785374671 -0.292970498838426 -0.0213107930928151 rpy=-1.5707963267949 1.52758843931606 1.5707963267949 -> xyz=0.1605 0.307 0.00085305 rpy=3.1416 -1.5708 0
- joint joint_6: origin xyz=-0.0914130137207118 0.180882427216801 0 rpy=3.14159265358979 0 -3.14159265358979 -> xyz=0 0.181 0 rpy=3.1416 0 3.1416
- joint joint_7: axis 0 0.999066684445606 -0.0431944444444357 -> 0 1 0; child end_efector -> EF; origin xyz=0 0.1621961599513 0.0168602146253252 rpy=0.0432078874788314 1.5707963267949 0 -> xyz=0 0.16219 -0.016 rpy=3.1416 -1.5708 0

Commit message: Add files via upload

File: robot_siad7n/urdf/robot_siad7n.urdf (robot description, URDF)
Before this commit: robot robot_siad7n, 8 links, 7 joints
Links:
- link EF: mass 9.59762719689291E-05 -> 9.5976E-05
- link link_1: mass 0.0117569497463589 -> 0.011757
- link link_2: mass 10.0552877935848 -> 10.055
- link link_3: mass 0.00843890832225914 -> 0.0084389
- link link_4: mass 6.45548607858182 -> 6.4555
- link link_5: mass 0.00287980676910192 -> 0.0028798
Joints:
- joint joint_4: limit lower=-1.3963 upper=4.5379 effort=0 velocity=0 -> lower=-4.5379 upper=1.3963 effort=0 velocity=0

Commit message: Add files via upload

File: robot_siad7n/urdf/robot_siad7n.urdf (robot description, URDF)
Before this commit: robot robot_siad7n, 8 links, 7 joints
Joints:
- removed joint join_3
- added joint joint_3: type prismatic, parent link_2, child link_3, origin xyz=3.4347E-05 0.3019 0.265 rpy=0 0 3.1416, axis 0 1 0, limit lower=0 upper=0.32 effort=100 velocity=10
- joint joint_4: limit lower=-4.5379 upper=1.3963 effort=0 velocity=0 -> lower=4.5379 upper=-1.3963 effort=0 velocity=0; origin xyz=0 -0.2426 0 rpy=3.1416 0 -1.5708 -> xyz=0 -0.2426 0 rpy=-3.1416 0 -1.5708

Commit message: Add files via upload

File: robot_siad7n/urdf/robot_siad7n.urdf (robot description, URDF)
Before this commit: robot robot_siad7n, 8 links, 7 joints
Links:
- link link_3: mass 0.0084389 -> 0.00843890832225914
- link link_4: mass 6.4555 -> 6.45548612950254
Joints:
- joint joint_1: origin xyz=0 0 0.1175 rpy=1.5708 0 0 -> xyz=0 0 0.1175 rpy=1.5708 0 1.5708
- joint joint_3: origin xyz=3.4347E-05 0.3019 0.265 rpy=0 0 3.1416 -> xyz=3.43471413583333E-05 0.301899975 0.265 rpy=0 0 3.14159265358979
- joint joint_4: limit lower=4.5379 upper=-1.3963 effort=0 velocity=0 -> lower=-4.5379 upper=1.3963 effort=0 velocity=0; origin xyz=0 -0.2426 0 rpy=-3.1416 0 -1.5708 -> xyz=0 -0.242600025 0 rpy=-3.14159265358979 0 -1.5707963267949
- joint joint_5: origin xyz=0.1605 0.307 0.00085305 rpy=3.1416 -1.5708 0 -> xyz=0.160499999999997 0.306999974999982 0.000853052852609892 rpy=3.14159265358979 -1.5707963267949 0
- joint joint_6: origin xyz=0 0.181 0 rpy=3.1416 0 3.1416 -> xyz=0 0.181000025000001 0 rpy=3.14159265358979 0 3.14159265358979
- joint joint_7: origin xyz=0 0.16219 -0.016 rpy=3.1416 -1.5708 0 -> xyz=0 0.16219 -0.016 rpy=3.1416 0 3.1416

Commit message: Add files via upload

File: robot_siad7n/urdf/robot_siad7n.urdf (robot description, URDF)
Before this commit: robot robot_siad7n, 8 links, 7 joints
Links:
- link EF: mass 9.5976E-05 -> 9.59762719689292E-05
- link base_link: mass 9.5605 -> 9.56045935245332
- link link_1: mass 0.011757 -> 0.0117569497463645
- link link_2: mass 10.055 -> 10.0552877935744
- link link_5: mass 0.0028798 -> 0.00287980676910192
- link link_6: mass 0.0020184 -> 0.00201842025658046
Joints:
- joint joint_1: origin xyz=0 0 0.1175 rpy=1.5708 0 1.5708 -> xyz=0 0 0.1175 rpy=1.5708 0 0
- joint joint_3: origin xyz=3.43471413583333E-05 0.301899975 0.265 rpy=0 0 3.14159265358979 -> xyz=3.4347E-05 0.3019 0.265 rpy=0 0 3.1416
- joint joint_4: origin xyz=0 -0.242600025 0 rpy=-3.14159265358979 0 -1.5707963267949 -> xyz=0 -0.2426 0 rpy=-3.1416 0 -1.5708
- joint joint_7: origin xyz=0 0.16219 -0.016 rpy=3.1416 0 3.1416 -> xyz=0 0.162188781523228 -0.0160000000000009 rpy=3.14159265358979 0 3.14159265358979

Commit message: Add files via upload

File: robot_siad7n/urdf/robot_siad7n.urdf (robot description, URDF)
Before this commit: robot robot_siad7n, 8 links, 7 joints
Joints:
- joint joint_3: limit lower=0 upper=0.32 effort=100 velocity=10 -> lower=-0.32 upper=0 effort=100 velocity=10
- joint joint_5: origin xyz=0.160499999999997 0.306999974999982 0.000853052852609892 rpy=3.14159265358979 -1.5707963267949 0 -> xyz=0.160499999999997 0.306999974999982 0.000853052852609892 rpy=0 -1.5707963267949 0

Commit message: Add files via upload

File: robot_siad7n/urdf/robot_siad7n.urdf (robot description, URDF)
Before this commit: robot robot_siad7n, 8 links, 7 joints
Joints:
- joint joint_3: axis 0 1 0 -> 0 -1 0; limit lower=-0.32 upper=0 effort=100 velocity=10 -> lower=0 upper=0.32 effort=100 velocity=10

Commit message: Add files via upload

File: robot_siad7n/urdf/robot_siad7n.urdf (robot description, URDF)
Before this commit: robot robot_siad7n, 8 links, 7 joints
Links:
- added link world
Joints:
- added joint world_joint: type fixed, parent world, child base_link, origin xyz=0.0 0.0 0.0 rpy=0.0 0.0 0.0
- joint joint_2: limit lower=-1.5708 upper=1.5708 effort=0 velocity=0 -> lower=-1.5708 upper=1.5708 effort=100 velocity=50
- joint joint_4: limit lower=-4.5379 upper=1.3963 effort=0 velocity=0 -> lower=-4.5379 upper=1.3963 effort=100 velocity=50
- joint joint_5: limit lower=0 upper=0.25 effort=0 velocity=0 -> lower=0 upper=0.25 effort=100 velocity=10
- joint joint_6: limit lower=-1.5708 upper=1.5708 effort=0 velocity=0 -> lower=-1.5708 upper=1.5708 effort=100 velocity=50
- joint joint_7: limit lower=-3.1416 upper=3.1416 effort=0 velocity=0 -> lower=-3.1416 upper=3.1416 effort=100 velocity=50
